File: Final Keyboard PCB/IEEE Keyboard Project.kicad_pcb (KiCad board)
At the start: 4 copper layers, 188.8 x 165.5 mm, 180 parts, among them J1 Conn_01x04_Socket, J2 Conn_01x04_Socket, P3 USB_C_Plug_USB2.0, P4 USB_C_Plug_USB2.0, SW1 SW_Push, SW2 SW_Push, SW3 SW_Push, SW4 SW_Push, SW5 SW_Nidec_CAS-120A1, U1 RP2354B, U2 RP2354B, U3 NCP1117-3.3_SOT223, U5 NCP1117-3.3_SOT223, Y2 ABM8-272-T3, Y5 ABM8-272-T3, Y6 ABM8-272-T3

Commit message: Update IEEE Keyboard Project.kicad_pcb
Routing:
- added copper zone on In1.Cu, net +3V3
- added copper zone on In2.Cu, net GND
Changed lines of the file:
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@@
+		)
+	)
+	(zone
+		(net "+3V3")
+		(layer "In1.Cu")
+		(hatch edge 0.5)
+		(priority 1)
+		(connect_pads
+			(clearance 0.1)
+		)
+		(min_thickness 0.25)
+		(fill
+			(thermal_gap 0.5)
+			(thermal_bridge_width 0.5)
+			(island_removal_mode 0)
+		)
+		(polygon
+			(pts
+				(xy 67.5 18) (xy 25 133.5) (xy 173 183.5) (xy 214 68)
+			)
+		)
+	)
+	(zone
+		(net "GND")
+		(layer "In2.Cu")
+		(hatch edge 0.5)
+		(connect_pads
+			(clearance 0.1)
+		)
+		(min_thickness 0.25)
+		(fill
+			(thermal_gap 0.5)
+			(thermal_bridge_width 0.5)
+			(island_removal_mode 0)
+		)
+		(polygon
+			(pts
+				(xy 67.5 18) (xy 25 133.5) (xy 173 183.5) (xy 214 68)
+			)
 		)
 	)

Commit message: Update IEEE Keyboard Project.kicad_pcb
Parts:
- moved R10 0.48 mm to (267.0, 228.5)
Changed lines of the file:
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@@
 	(footprint "Resistor_SMD:R_0402_1005Metric"
 		(layer "F.Cu")
-		(at 267.49 228.5)
+		(at 267.01 228.5)
 		(descr "Resistor SMD 0402 (1005 Metric), square (rectangular) end terminal, IPC-7351 nominal, (Body size source: IPC-SM-782 page 72, https://www.pcb-3d.com/wordpress/wp-content/uploads/ipc-sm-782a_amendment_1_and_2.pdf)")
 		(tags "resistor")
