File: IEEE Keyboard Project.kicad_pcb (KiCad board)
At the start: 4 copper layers, 188.8 x 165.5 mm, 180 parts, among them J1 Conn_01x04_Socket, J2 Conn_01x04_Socket, P3 USB_C_Plug_USB2.0, P4 USB_C_Plug_USB2.0, SW1 SW_Push, SW2 SW_Push, SW3 SW_Push, SW4 SW_Push, SW5 SW_Nidec_CAS-120A1, U1 RP2354B, U2 RP2354B, U3 NCP1117-3.3_SOT223, U5 NCP1117-3.3_SOT223, Y2 ABM8-272-T3, Y5 ABM8-272-T3, Y6 ABM8-272-T3

Commit message: Update IEEE Keyboard Project.kicad_pcb
Routing:
- net COL4: track 0.00 -> 85.4 mm
- net COL5: track 0.00 -> 85.2 mm
- net COL0: track 0.00 -> 66.5 mm
- net COL2: track 0.00 -> 63.6 mm
- net COL1: track 0.00 -> 62.9 mm
- net COL3: track 0.00 -> 62.6 mm
- net COL6: track 0.00 -> 20.5 mm

Commit message: Update IEEE Keyboard Project.kicad_pcb
Parts:
- moved R2 2.53 mm to (188.0, 105.5), turned to 180 degrees
Routing:
- net ROW0: track 0.00 -> 126.2 mm
- net ROW1: track 0.00 -> 122.0 mm
- net ROW2: track 0.00 -> 118.3 mm
- net Net-(D1-A): track 0.00 -> 14.3 mm
- net Net-(D5-A): track 0.00 -> 12.4 mm
- net Net-(D3-A): track 0.00 -> 11.9 mm
- net Net-(D2-A): track 0.00 -> 11.3 mm
- net Net-(D6-A): track 0.00 -> 11.0 mm
- net Net-(D4-A): track 0.00 -> 11.0 mm
- net COL5: track 85.2 -> 88.5 mm
- net COL0: track 66.5 -> 65.6 mm
