File: .history/IEEE Keyboard Project.kicad_pcb (KiCad board)
At the start: 4 copper layers, 188.8 x 165.5 mm, 180 parts, among them J1 Conn_01x04_Socket, J2 Conn_01x04_Socket, P3 USB_C_Plug_USB2.0, P4 USB_C_Plug_USB2.0, SW1 SW_Push, SW2 SW_Push, SW3 SW_Push, SW4 SW_Push, SW5 SW_Nidec_CAS-120A1, U1 RP2354B, U2 RP2354B, U3 NCP1117-3.3_SOT223, U5 NCP1117-3.3_SOT223, Y2 ABM8-272-T3, Y5 ABM8-272-T3, Y6 ABM8-272-T3

Commit message: Update IEEE Keyboard Project.kicad_pcb
Parts:
- moved R2 16.1 mm to (172.0, 107.0), turned to 90 degrees
- moved C26 9.32 mm to (170.4, 101.5)
- moved C19 9.32 mm to (169.5, 103.0)
- moved R5 6.52 mm to (173.5, 101.5)
Routing:
- net ROW3: track 0.00 -> 162.6 mm
- net ROW2: track 118.3 -> 134.0 mm
