File: .history/IEEE Keyboard Project.kicad_pcb (KiCad board)
At the start: 4 copper layers, 188.8 x 165.5 mm, 180 parts, among them J1 Conn_01x04_Socket, J2 Conn_01x04_Socket, P3 USB_C_Plug_USB2.0, P4 USB_C_Plug_USB2.0, SW1 SW_Push, SW2 SW_Push, SW3 SW_Push, SW4 SW_Push, SW5 SW_Nidec_CAS-120A1, U1 RP2354B, U2 RP2354B, U3 NCP1117-3.3_SOT223, U5 NCP1117-3.3_SOT223, Y2 ABM8-272-T3, Y5 ABM8-272-T3, Y6 ABM8-272-T3

Commit message: Update IEEE Keyboard Project.kicad_pcb
Routing:
- net ROW4: track 0.00 -> 51.3 mm
- net Net-(D26-A): track 0.00 -> 8.14 mm
- net Net-(D14-A): track 0.00 -> 8.05 mm
- net Net-(D18-A): track 0.00 -> 8.04 mm
- net Net-(D16-A): track 0.00 -> 8.02 mm
- net Net-(D15-A): track 0.00 -> 7.99 mm
- net Net-(D17-A): track 0.00 -> 7.96 mm
- net Net-(D25-A): track 0.00 -> 7.85 mm
- net Net-(D13-A): track 0.00 -> 7.61 mm
- net Net-(D28-A): track 0.00 -> 7.60 mm
Changed lines of the file:
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@@
+	)
+	(segment
+		(start 134.37286 153.34786)
+		(end 134.37286 147.545752)
+		(width 0.2)
+		(layer "B.Cu")
+		(net "Net-(D26-A)")
+	)
+	(segment
+		(start 136.025 155)
+		(end 134.37286 153.34786)
+		(width 0.2)
+		(layer "B.Cu")
+		(net "Net-(D26-A)")
 	)
 	(segment
@@
 	)
 	(segment
+		(start 136.525 156.975)
+		(end 133.5125 159.9875)
+		(width 0.2)
+		(layer "B.Cu")
+		(net "ROW4")
+	)
+	(segment
+		(start 136.525 155)
+		(end 136.525 156.975)
+		(width 0.2)
+		(layer "B.Cu")
+		(net "ROW4")
+	)
+	(segment
+		(start 153.76991 165.4875)
+		(end 154.525 164.73241)
+		(width 0.2)
+		(layer "B.Cu")
+		(net "ROW4")
+	)
+	(segment
+		(start 139.0125 165.4875)
+		(end 153.76991 165.4875)
+		(width 0.2)
+		(layer "B.Cu")
+		(net "ROW4")
+	)
+	(segment
+		(start 139.0125 165.4875)
+		(end 139.025 165.5)
+		(width 0.2)
+		(layer "B.Cu")
+		(net "ROW4")
+	)
+	(segment
+		(start 118.525 145)
+		(end 133.5125 159.9875)
+		(width 0.2)
+		(layer "B.Cu")
+		(net "ROW4")
+	)
+	(segment
+		(start 154.525 164.73241)
+		(end 154.525 164.5)
+		(width 0.2)
+		(layer "B.Cu")
+		(net "ROW4")
+	)
+	(segment
+		(start 133.5125 159.9875)
+		(end 139.0125 165.4875)
+		(width 0.2)
+		(layer "B.Cu")
+		(net "ROW4")
+	)
+	(segment
 		(start 75.5 43.332555)
 		(end 75.5 47.5)
@@
 	)
 	(segment
+		(start 115.75 95.5)
+		(end 114.5 94.25)
+		(width 0.2)
+		(layer "B.Cu")
+		(net "Net-(D16-A)")
+	)
+	(segment
+		(start 114.5 94.25)
+		(end 114.5 87.999999)
+		(width 0.2)
+		(layer "B.Cu")
+		(net "Net-(D16-A)")
+	)
+	(segment
 		(start 145 73)
 		(end 144 73)
@@
 	)
 	(segment
+		(start 56.5 87)
+		(end 55.475285 85.975285)
+		(width 0.2)
+		(layer "B.Cu")
+		(net "Net-(D13-A)")
+	)
+	(segment
+		(start 55.475285 85.975285)
+		(end 55.475285 79.817431)
+		(width 0.2)
+		(layer "B.Cu")
+		(net "Net-(D13-A)")
+	)
+	(segment
+		(start 149 118)
+		(end 147.514864 116.514864)
+		(width 0.2)
+		(layer "B.Cu")
+		(net "Net-(D18-A)")
+	)
+	(segment
+		(start 147.514864 116.514864)
+		(end 147.514864 110.572621)
+		(width 0.2)
+		(layer "B.Cu")
+		(net "Net-(D18-A)")
+	)
+	(segment
+		(start 96.025 93.5)
+		(end 94.509888 91.984888)
+		(width 0.2)
+		(layer "B.Cu")
+		(net "Net-(D15-A)")
+	)
+	(segment
+		(start 94.509888 91.984888)
+		(end 94.509888 86.136233)
+		(width 0.2)
+		(layer "B.Cu")
+		(net "Net-(D15-A)")
+	)
+	(segment
+		(start 154.025 158.044943)
+		(end 154.835915 157.234028)
+		(width 0.2)
+		(layer "B.Cu")
+		(net "Net-(D28-A)")
+	)
+	(segment
+		(start 154.025 164.5)
+		(end 154.025 158.044943)
+		(width 0.2)
+		(layer "B.Cu")
+		(net "Net-(D28-A)")
+	)
+	(segment
+		(start 75 94)
+		(end 73.664221 92.664221)
+		(width 0.2)
+		(layer "B.Cu")
+		(net "Net-(D14-A)")
+	)
+	(segment
+		(start 73.664221 92.664221)
+		(end 73.664221 86.5)
+		(width 0.2)
+		(layer "B.Cu")
+		(net "Net-(D14-A)")
+	)
+	(segment
 		(start 72.5 50)
 		(end 72.087462 49.587462)
@@
 		(layer "B.Cu")
 		(net "Net-(D2-A)")
+	)
+	(segment
+		(start 118.025 145)
+		(end 117.014864 143.989864)
+		(width 0.2)
+		(layer "B.Cu")
+		(net "Net-(D25-A)")
+	)
+	(segment
+		(start 117.014864 143.989864)
+		(end 117.014864 137.572621)
+		(width 0.2)
+		(layer "B.Cu")
+		(net "Net-(D25-A)")
+	)
+	(segment
+		(start 132.25 108)
+		(end 130.624221 106.374221)
+		(width 0.2)
+		(layer "B.Cu")
+		(net "Net-(D17-A)")
+	)
+	(segment
+		(start 130.624221 106.374221)
+		(end 130.624221 100.713489)
+		(width 0.2)
+		(layer "B.Cu")
+		(net "Net-(D17-A)")
 	)
 	(zone
@@
 		(connect_pads
 			(clearance 0.1)
+		)
+		(min_thickness 0.25)
+		(fill yes
+			(thermal_gap 0.5)
+			(thermal_bridge_width 0.5)
+			(island_removal_mode 0)
+		)
+		(polygon
+			(pts
+				(xy 67.5 18) (xy 25 133.5) (xy 173 183.5) (xy 214 68)
+			)
+		)
+	)
+	(zone
+		(net "+3V3")
+		(layer "In1.Cu")
+		(name "3V3")
+		(hatch edge 0.5)
+		(priority 4)
+		(connect_pads
+			(clearance 0.1)

Commit message: Update IEEE Keyboard Project.kicad_pcb
Parts:
- moved SW5 40.0 mm to (181.9, 89.4)
- moved R1 31.4 mm to (186.4, 74.7)
- moved C2 22.8 mm to (190.8, 82.1)
- moved C6 22.8 mm to (192.5, 78.0)
- moved U3 22.8 mm to (198.5, 83.0)
- moved R3 16.2 mm to (200.3, 75.5)
- moved R4 15.9 mm to (197.5, 75.0)
- moved C32 6.98 mm to (190.0, 106.7), turned to -90 degrees
- moved C23 6.44 mm to (187.5, 106.2), turned to -90 degrees
- moved C13 3.97 mm to (183.4, 104.8), turned to -110 degrees
- moved C28 3.36 mm to (185.4, 105.7), turned to -90 degrees
Routing:
- net Net-(D27-A): track 0.00 -> 9.51 mm
- net VBUS: track 0.00 -> 4.70 mm
- net GND: vias 0 -> 30
- net +3V3: vias 0 -> 16
